File: uv1.sch (KiCad schematic (older format))
At the start: 15 parts, among them J1 Conn_02x06_Odd_Even, J2 Conn_01x02, U1 TC7106, U2 LCD-A2X1C50TR

Commit message: Display DE151 Sensor connector 2x 2x2 male
Parts:
- removed J1: Conn_02x06_Odd_Even, Connector_PinSocket_2.54mm:PinSocket_2x06_P2.54mm_Horizontal, symbol Connector_Generic:Conn_02x06_Odd_Even
- removed R5: 2.2k, Resistor_SMD:R_1206_3216Metric, symbol Device:R
- removed U2: LCD-A2X1C50TR, uv1:LCD-A2X1C50TR, symbol uv1:LCD-A2X1C50TR
- added D1: LM285D-1.2, Package_SO:SOIC-8_3.9x4.9mm_P1.27mm, symbol Reference_Voltage:LM285D-1.2
- added J1, J3: Conn_02x02_Odd_Even, Connector_PinHeader_2.54mm:PinHeader_2x02_P2.54mm_Horizontal, symbol Connector_Generic:Conn_02x02_Odd_Even
- added SW1: SW_Push, uv1:MEC_3FTH9, symbol Switch:SW_Push
- added U2: DE151-RS-20, uv1:DE151-RS-20, symbol uv1:DE151-RS-20
- C1: footprint Capacitor_SMD:C_1206_3216Metric -> Capacitor_THT:C_Rect_L7.0mm_W2.5mm_P5.00mm
- R4: value 24k -> 6.8k
- RV1: value 1k -> 20k
Connections:
- net labels added: LCD_-, LCD_1BC, LCD_2A, LCD_2B, LCD_2C, LCD_2D, LCD_2E, LCD_2F, LCD_2G, LCD_3A, LCD_3B, LCD_3C, LCD_3D, LCD_3E, LCD_3F, LCD_3G, LCD_4A, LCD_4B, LCD_4C, LCD_4D, LCD_4E, LCD_4F, LCD_4G, LCD_BP, LCD_DP3
- net labels removed: 1BC, 2A, 2B, 2C, 2D, 2E, 2F, 2G, 3A, 3B, 3C, 3D, 3E, 3F, 3G, BP
- wire segments 92 -> 125
- no-connect marks 15 -> 2
Other:
- note added: "C1 polypropylene or polyester\nC2, C4 mylar\nC3, C5 ceramic"
- note added: "TC7106 digits are numbered right to left\nDE151 digits are numbered left to right"
- note added: "Vref should be 420 +/- 150 mV\nto give FS of 199mMED/hr +/- 30%\n**TODO Change V reference to LM185"
- note removed: "Vref should be 420 +/- 150 mV\nto give FS of 199mMED/hr +/- 30%\n**TODO: include a bandgap reference"

Commit message: DE115 LCD with new footprint + 3D
Parts:
- removed U2: DE151-RS-20, uv1:DE151-RS-20, symbol uv1:DE151-RS-20
- added U2: DE115-RS-20, uv1:DE115-RS-20, symbol uv1:DE115-RS-20
Connections:
- net labels added: LCD_1A, LCD_1B, LCD_1C, LCD_1D, LCD_1E, LCD_1F, LCD_1G
- net labels removed: LCD_4A, LCD_4B, LCD_4C, LCD_4D, LCD_4E, LCD_4F, LCD_4G
- wire segments 125 -> 124
Changed lines of the file:
@@
 	1700 6350 2000 6350
 Text Label 5300 2300 2    50   ~ 0
-LCD_3A
+LCD_2A
 Text Label 5300 2400 2    50   ~ 0
-LCD_3B
+LCD_2B
 Text Label 5300 2500 2    50   ~ 0
-LCD_3C
+LCD_2C
 Text Label 5300 2600 2    50   ~ 0
-LCD_3D
+LCD_2D
 Text Label 5300 2700 2    50   ~ 0
-LCD_3E
+LCD_2E
 Text Label 5300 2800 2    50   ~ 0
-LCD_3F
+LCD_2F
 Text Label 5300 2900 2    50   ~ 0
-LCD_3G
+LCD_2G
 Text Label 5300 3000 2    50   ~ 0
-LCD_2A
+LCD_1A
 Text Label 5300 3100 2    50   ~ 0
-LCD_2B
+LCD_1B
 Text Label 5300 3200 2    50   ~ 0
-LCD_2C
+LCD_1C
 Text Label 5300 3300 2    50   ~ 0
-LCD_2D
+LCD_1D
 Text Label 5300 3400 2    50   ~ 0
-LCD_2E
+LCD_1E
 Text Label 5300 3500 2    50   ~ 0
-LCD_2F
+LCD_1F
 Text Label 5300 3600 2    50   ~ 0
-LCD_2G
+LCD_1G
 Text Label 5300 3700 2    50   ~ 0
 LCD_BP
@@
 LCD_BP
 Text Label 7600 2100 0    50   ~ 0
+LCD_1A
+Text Label 7600 2200 0    50   ~ 0
+LCD_1B
+Text Label 7600 2300 0    50   ~ 0
+LCD_1C
+Text Label 7600 2400 0    50   ~ 0
+LCD_1D
+Text Label 7600 2500 0    50   ~ 0
+LCD_1E
+Text Label 7600 2600 0    50   ~ 0
+LCD_1F
+Text Label 7600 2700 0    50   ~ 0
+LCD_1G
+Text Label 7600 2800 0    50   ~ 0
+LCD_BP
+Text Label 7600 2900 0    50   ~ 0
 LCD_2A
-Text Label 7600 2200 0    50   ~ 0
+Text Label 7600 3000 0    50   ~ 0
 LCD_2B
-Text Label 7600 2300 0    50   ~ 0
+Text Label 7600 3100 0    50   ~ 0
 LCD_2C
-Text Label 7600 2400 0    50   ~ 0
+Text Label 7600 3200 0    50   ~ 0
 LCD_2D
-Text Label 7600 2500 0    50   ~ 0
+Text Label 7600 3300 0    50   ~ 0
 LCD_2E
-Text Label 7600 2600 0    50   ~ 0
+Text Label 7600 3400 0    50   ~ 0
 LCD_2F
-Text Label 7600 2700 0    50   ~ 0
+Text Label 7600 3500 0    50   ~ 0
 LCD_2G
-Text Label 7600 2800 0    50   ~ 0
-LCD_BP
-Text Label 7600 2900 0    50   ~ 0
-LCD_3A
-Text Label 7600 3000 0    50   ~ 0
-LCD_3B
-Text Label 7600 3100 0    50   ~ 0
-LCD_3C
-Text Label 7600 3200 0    50   ~ 0
-LCD_3D
-Text Label 7600 3300 0    50   ~ 0
-LCD_3E
-Text Label 7600 3400 0    50   ~ 0
-LCD_3F
-Text Label 7600 3500 0    50   ~ 0
-LCD_3G
 Text Label 9550 2100 2    50   ~ 0
 LCD_DP3
 Text Label 9550 2200 2    50   ~ 0
-LCD_4A
+LCD_3A
 Text Label 9550 2300 2    50   ~ 0
-LCD_4B
+LCD_3B
 Text Label 9550 2400 2    50   ~ 0
-LCD_4C
+LCD_3C
 Text Label 9550 2500 2    50   ~ 0
-LCD_4D
+LCD_3D
 Text Label 9550 2600 2    50   ~ 0
-LCD_4E
+LCD_3E
 Text Label 9550 2700 2    50   ~ 0
-LCD_4F
+LCD_3F
 Text Label 9550 2800 2    50   ~ 0
-LCD_4G
+LCD_3G
 Text Label 9550 2900 2    50   ~ 0
 LCD_BP
@@
 Text Label 9550 3400 2    50   ~ 0
 LCD_1BC
-Text Label 9550 3500 2    50   ~ 0
-LCD_BP
 Wire Wire Line
 	7600 2000 7900 2000
@@
 	5300 3900 4900 3900
 Text Label 5300 1600 2    50   ~ 0
-LCD_4A
+LCD_3A
 Text Label 5300 1700 2    50   ~ 0
-LCD_4B
+LCD_3B
 Text Label 5300 1800 2    50   ~ 0
-LCD_4C
+LCD_3C
 Text Label 5300 1900 2    50   ~ 0
-LCD_4D
+LCD_3D
 Text Label 5300 2000 2    50   ~ 0
-LCD_4E
+LCD_3E
 Text Label 5300 2100 2    50   ~ 0
-LCD_4F
+LCD_3F
 Text Label 5300 2200 2    50   ~ 0
-LCD_4G
+LCD_3G
 Wire Wire Line
 	4900 1600 5300 1600
@@
 Wire Wire Line
 	9100 3400 9550 3400
-Wire Wire Line
-	9100 3500 9550 3500
 $Comp
 L uv1:TC7106 U1
@@
 $EndComp
 $Comp
-L uv1:DE151-RS-20 U2
-U 1 1 5BBB0B28
+L uv1:DE115-RS-20 U2
+U 1 1 5BBEEF2D
 P 8500 2500
 F 0 "U2" H 8500 3767 50  0000 C CNN
-F 1 "DE151-RS-20" H 8500 3676 50  0000 C CNN
-F 2 "uv1:DE151-RS-20" H 8500 1200 50  0001 C CNN
+F 1 "DE115-RS-20" H 8500 3676 50  0000 C CNN
+F 2 "uv1:DE115-RS-20" H 8500 1200 50  0001 C CNN
 F 3 "" H 8300 2700 50  0001 C CNN
 	1    8500 2500

Commit message: 2x7 sensor connector
Parts:
- removed J1, J3: Conn_02x02_Odd_Even, Connector_PinHeader_2.54mm:PinHeader_2x02_P2.54mm_Horizontal, symbol Connector_Generic:Conn_02x02_Odd_Even
- added J1: Conn_02x07_Odd_Even, Connector_PinSocket_2.54mm:PinSocket_2x07_P2.54mm_Horizontal, symbol Connector_Generic:Conn_02x07_Odd_Even
Connections:
- no-connect marks 2 -> 9
Other:
- note added: "TC7106 digits are numbered right to left\nDE115 digits are numbered left to right"
- note removed: "TC7106 digits are numbered right to left\nDE151 digits are numbered left to right"
Changed lines of the file:
@@
 Wire Wire Line
 	1450 2550 1650 2550
-Wire Wire Line
-	1650 1450 1650 2050
-Wire Wire Line
-	2150 1450 2150 2050
-$Comp
-L Connector_Generic:Conn_02x02_Odd_Even J1
-U 1 1 5BBE1B4E
-P 1850 2050
-F 0 "J1" H 1900 2267 50  0000 C CNN
-F 1 "Conn_02x02_Odd_Even" H 1900 2176 50  0000 C CNN
-F 2 "Connector_PinHeader_2.54mm:PinHeader_2x02_P2.54mm_Horizontal" H 1850 2050 50  0001 C CNN
-F 3 "~" H 1850 2050 50  0001 C CNN
-	1    1850 2050
-	1    0    0    -1
-$EndComp
-Wire Wire Line
-	1650 2050 1650 2150
-Connection ~ 1650 2050
-Wire Wire Line
-	2150 2050 2150 2150
-Connection ~ 2150 2050
-$Comp
-L Connector_Generic:Conn_02x02_Odd_Even J3
-U 1 1 5BBEA97D
-P 1850 2550
-F 0 "J3" H 1900 2767 50  0000 C CNN
-F 1 "Conn_02x02_Odd_Even" H 1900 2676 50  0000 C CNN
-F 2 "Connector_PinHeader_2.54mm:PinHeader_2x02_P2.54mm_Horizontal" H 1850 2550 50  0001 C CNN
-F 3 "~" H 1850 2550 50  0001 C CNN
-	1    1850 2550
-	1    0    0    -1
-$EndComp
 Text Notes 5600 1950 0    50   ~ 0
-TC7106 digits are numbered right to left\nDE151 digits are numbered left to right
+TC7106 digits are numbered right to left\nDE115 digits are numbered left to right
 Text Notes 2100 5000 2    50   ~ 0
 C1 polypropylene or polyester\nC2, C4 mylar\nC3, C5 ceramic
@@
 	1    0    0    -1
 $EndComp
+$Comp
+L Connector_Generic:Conn_02x07_Odd_Even J1
+U 1 1 5BBEC155
+P 1850 2350
+F 0 "J1" H 1900 2867 50  0000 C CNN
+F 1 "Conn_02x07_Odd_Even" H 1900 2776 50  0000 C CNN
+F 2 "Connector_PinSocket_2.54mm:PinSocket_2x07_P2.54mm_Horizontal" H 1850 2350 50  0001 C CNN
+F 3 "~" H 1850 2350 50  0001 C CNN
+	1    1850 2350
+	1    0    0    -1
+$EndComp
+Wire Wire Line
+	1650 1450 1650 2050
+Wire Wire Line
+	2150 1450 2150 2050
+Wire Wire Line
+	1650 2150 1650 2050
+Connection ~ 1650 2050
+Wire Wire Line
+	2150 2050 2150 2150
+Connection ~ 2150 2050
+NoConn ~ 2150 2250
+NoConn ~ 2150 2350
+NoConn ~ 2150 2450
+NoConn ~ 1650 2450
+NoConn ~ 1650 2350
+NoConn ~ 1650 2250
+NoConn ~ 5800 1900
 $EndSCHEMATC

Commit message: Fully routed by autorouter + tweaks
Parts:
- removed J2: Conn_01x02, Connector_PinHeader_2.54mm:PinHeader_1x02_P2.54mm_Vertical, symbol Connector_Generic:Conn_01x02
- added J2: - +, TestPoint:TestPoint_2Pads_Pitch2.54mm_Drill0.8mm, symbol Connector:TestPoint_2Pole
- added JP1: Jumper_NO_Small, Connector_PinHeader_1.27mm:PinHeader_1x02_P1.27mm_Vertical, symbol Device:Jumper_NO_Small
- added R5: 470k, Resistor_SMD:R_1206_3216Metric, symbol Device:R
- added U3: 74AHC1G04, Package_TO_SOT_SMD:SOT-23-5, symbol 74xGxx:74AHC1G04
- added U4, U5: 74HC157, Package_SO:TSSOP-16_4.4x5mm_P0.65mm, symbol 74xx:74LS157
- U1: footprint Package_DIP:DIP-40_W15.24mm -> Package_QFP:TQFP-44_10x10mm_P0.8mm
Connections:
- net labels added: +BATT, -BATT, DIGIT3_EN, GNDD, MUX_3A, MUX_3B, MUX_3C, MUX_3D, MUX_3E, MUX_3F, MUX_3G, VCC, VDD, VSS
- net labels removed: +9V, 0V
- wire segments 124 -> 163
- no-connect marks 9 -> 6
Other:
- note added: "0.1"
- note added: "12/10/2018"
- note added: "Main board"
- note added: "UV radiometer"
- note added: "VREF+ should be 420 +/- 150 mV\nto give FS of 199mMED/hr +/- 30%\n**TODO Change V reference to LM185"
- note removed: "Vref should be 420 +/- 150 mV\nto give FS of 199mMED/hr +/- 30%\n**TODO Change V reference to LM185"

Commit message: Decoupling caps added
Parts:
- added C6, C7, C8, C9: C, symbol Device:C
Connections:
- wire segments 163 -> 171
Changed lines of the file:
@@
 L power:PWR_FLAG #FLG0101
 U 1 1 5BAB272C
-P 1100 6000
-F 0 "#FLG0101" H 1100 6075 50  0001 C CNN
-F 1 "PWR_FLAG" H 1100 6174 50  0000 C CNN
-F 2 "" H 1100 6000 50  0001 C CNN
-F 3 "~" H 1100 6000 50  0001 C CNN
-	1    1100 6000
+P 1100 5850
+F 0 "#FLG0101" H 1100 5925 50  0001 C CNN
+F 1 "PWR_FLAG" H 1100 6024 50  0000 C CNN
+F 2 "" H 1100 5850 50  0001 C CNN
+F 3 "~" H 1100 5850 50  0001 C CNN
+	1    1100 5850
 	1    0    0    -1
 $EndComp
@@
 L power:PWR_FLAG #FLG0102
 U 1 1 5BAB27DC
-P 1100 6500
-F 0 "#FLG0102" H 1100 6575 50  0001 C CNN
-F 1 "PWR_FLAG" H 1100 6674 50  0000 C CNN
-F 2 "" H 1100 6500 50  0001 C CNN
-F 3 "~" H 1100 6500 50  0001 C CNN
-	1    1100 6500
-	1    0    0    -1
-$EndComp
-Wire Wire Line
-	1100 6000 1500 6000
+P 1100 6350
+F 0 "#FLG0102" H 1100 6425 50  0001 C CNN
+F 1 "PWR_FLAG" H 1100 6524 50  0000 C CNN
+F 2 "" H 1100 6350 50  0001 C CNN
+F 3 "~" H 1100 6350 50  0001 C CNN
+	1    1100 6350
+	1    0    0    -1
+$EndComp
+Wire Wire Line
+	1100 5850 1500 5850
 Text Label 4900 2300 2    50   ~ 0
 LCD_2A
@@
 	4900 3800 4500 3800
 Wire Wire Line
-	1500 5950 1500 6000
-Connection ~ 1500 6000
+	1500 5800 1500 5850
+Connection ~ 1500 5850
 Text Notes 4550 6450 0    50   ~ 0
 VREF+ should be 420 +/- 150 mV\nto give FS of 199mMED/hr +/- 30%\n**TODO Change V reference to LM185
@@
 $EndComp
 Wire Wire Line
-	4500 4350 5250 4350
+	4500 4350 4650 4350
 Wire Wire Line
 	5250 4400 5250 4350
@@
 Main board
 Wire Wire Line
-	1850 6000 1850 6050
-Wire Wire Line
-	1500 6500 1850 6500
-Wire Wire Line
-	1850 6500 1850 6450
+	1850 5850 1850 5900
+Wire Wire Line
+	1500 6350 1850 6350
+Wire Wire Line
+	1850 6350 1850 6300
 $Comp
 L Connector:TestPoint_2Pole J2
 U 1 1 5BC17FBC
-P 1850 6250
-F 0 "J2" V 1804 6308 50  0000 L CNN
-F 1 "-  +" V 1895 6308 50  0000 L CNN
-F 2 "TestPoint:TestPoint_2Pads_Pitch2.54mm_Drill0.8mm" H 1850 6250 50  0001 C CNN
-F 3 "~" H 1850 6250 50  0001 C CNN
-	1    1850 6250
+P 1850 6100
+F 0 "J2" V 1804 6158 50  0000 L CNN
+F 1 "-  +" V 1895 6158 50  0000 L CNN
+F 2 "TestPoint:TestPoint_2Pads_Pitch2.54mm_Drill0.8mm" H 1850 6100 50  0001 C CNN
+F 3 "~" H 1850 6100 50  0001 C CNN
+	1    1850 6100
 	0    1    1    0
 $EndComp
@@
 L power:+BATT #PWR06
 U 1 1 5BC901A3
-P 1500 5950
-F 0 "#PWR06" H 1500 5800 50  0001 C CNN
-F 1 "+BATT" H 1515 6123 50  0000 C CNN
-F 2 "" H 1500 5950 50  0001 C CNN
-F 3 "" H 1500 5950 50  0001 C CNN
-	1    1500 5950
+P 1500 5800
+F 0 "#PWR06" H 1500 5650 50  0001 C CNN
+F 1 "+BATT" H 1515 5973 50  0000 C CNN
+F 2 "" H 1500 5800 50  0001 C CNN
+F 3 "" H 1500 5800 50  0001 C CNN
+	1    1500 5800
 	1    0    0    -1
 $EndComp
@@
 L power:+BATT #PWR015
 U 1 1 5BC90399
-P 7950 1350
-F 0 "#PWR015" H 7950 1200 50  0001 C CNN
-F 1 "+BATT" H 7965 1523 50  0000 C CNN
-F 2 "" H 7950 1350 50  0001 C CNN
-F 3 "" H 7950 1350 50  0001 C CNN
-	1    7950 1350
+P 7950 1150
+F 0 "#PWR015" H 7950 1000 50  0001 C CNN
+F 1 "+BATT" H 7965 1323 50  0000 C CNN
+F 2 "" H 7950 1150 50  0001 C CNN
+F 3 "" H 7950 1150 50  0001 C CNN
+	1    7950 1150
 	1    0    0    -1
 $EndComp
@@
 L power:+BATT #PWR017
 U 1 1 5BC903FA
-P 7950 3900
-F 0 "#PWR017" H 7950 3750 50  0001 C CNN
-F 1 "+BATT" H 7965 4073 50  0000 C CNN
-F 2 "" H 7950 3900 50  0001 C CNN
-F 3 "" H 7950 3900 50  0001 C CNN
-	1    7950 3900
+P 7950 3800
+F 0 "#PWR017" H 7950 3650 50  0001 C CNN
+F 1 "+BATT" H 7965 3973 50  0000 C CNN
+F 2 "" H 7950 3800 50  0001 C CNN
+F 3 "" H 7950 3800 50  0001 C CNN
+	1    7950 3800
 	1    0    0    -1
 $EndComp
@@
 L power:-BATT #PWR07
 U 1 1 5BC9044D
-P 1500 6500
-F 0 "#PWR07" H 1500 6350 50  0001 C CNN
-F 1 "-BATT" H 1515 6673 50  0000 C CNN
-F 2 "" H 1500 6500 50  0001 C CNN
-F 3 "" H 1500 6500 50  0001 C CNN
-	1    1500 6500
-	1    0    0    -1
+P 1500 6350
+F 0 "#PWR07" H 1500 6200 50  0001 C CNN
+F 1 "-BATT" H 1515 6523 50  0000 C CNN
+F 2 "" H 1500 6350 50  0001 C CNN
+F 3 "" H 1500 6350 50  0001 C CNN
+	1    1500 6350
+	-1   0    0    1
 $EndComp
 $Comp
@@
 F 3 "" H 5800 5700 50  0001 C CNN
 	1    5800 5700
-	1    0    0    -1
+	-1   0    0    1
 $EndComp
 $Comp
@@
 Connection ~ 1450 7350
 Wire Wire Line
-	1500 6000 1850 6000
+	1500 5850 1850 5850
 $Comp
 L power:GNDD #PWR0101
@@
 Wire Wire Line
 	6950 5200 7450 5200
-Connection ~ 1500 6500
-Wire Wire Line
-	1100 6500 1500 6500
+Connection ~ 1500 6350
+Wire Wire Line
+	1100 6350 1500 6350
+$Comp
+L Device:C C7
+U 1 1 5BC6470D
+P 8350 3900
+F 0 "C7" V 8098 3900 50  0000 C CNN
+F 1 "C" V 8189 3900 50  0000 C CNN
+F 2 "" H 8388 3750 50  0001 C CNN
+F 3 "~" H 8350 3900 50  0001 C CNN
+	1    8350 3900
+	0    1    1    0
+$EndComp
+$Comp
+L power:GNDD #PWR010
+U 1 1 5BC6D39A
+P 8550 3900
+F 0 "#PWR010" H 8550 3650 50  0001 C CNN
+F 1 "GNDD" H 8554 3745 50  0000 C CNN
+F 2 "" H 8550 3900 50  0001 C CNN
+F 3 "" H 8550 3900 50  0001 C CNN
+	1    8550 3900
+	1    0    0    -1
+$EndComp
+Wire Wire Line
+	8500 3900 8550 3900
+Wire Wire Line
+	8200 3900 7950 3900
+Wire Wire Line
+	7950 3900 7950 3800
+Connection ~ 7950 3900
+Wire Wire Line
+	7950 1150 7950 1200
+Wire Wire Line
+	7950 1200 8150 1200
+Connection ~ 7950 1200
+Wire Wire Line
+	7950 1200 7950 1350
+$Comp
+L Device:C C6
+U 1 1 5BCC7623
+P 8300 1200
+F 0 "C6" V 8048 1200 50  0000 C CNN
+F 1 "C" V 8139 1200 50  0000 C CNN
+F 2 "" H 8338 1050 50  0001 C CNN
+F 3 "~" H 8300 1200 50  0001 C CNN
+	1    8300 1200
+	0    1    1    0
+$EndComp
+$Comp
+L power:GNDD #PWR019
+U 1 1 5BCD099F
+P 8600 1200
+F 0 "#PWR019" H 8600 950 50  0001 C CNN
+F 1 "GNDD" H 8604 1045 50  0000 C CNN
+F 2 "" H 8600 1200 50  0001 C CNN
+F 3 "" H 8600 1200 50  0001 C CNN
+	1    8600 1200
+	1    0    0    -1
+$EndComp
+Wire Wire Line
+	8600 1200 8450 1200
+$Comp
+L Device:C C8
+U 1 1 5BCECC23
+P 4650 4500
+F 0 "C8" H 4765 4546 50  0000 L CNN
+F 1 "C" H 4765 4455 50  0000 L CNN
+F 2 "" H 4688 4350 50  0001 C CNN
+F 3 "~" H 4650 4500 50  0001 C CNN
+	1    4650 4500
+	1    0    0    -1
+$EndComp
+Connection ~ 4650 4350
+Wire Wire Line
+	4650 4350 5250 4350
+$Comp
+L power:-BATT #PWR020
+U 1 1 5BCECDF3
+P 4650 4650
+F 0 "#PWR020" H 4650 4500 50  0001 C CNN
+F 1 "-BATT" H 4665 4823 50  0000 C CNN
+F 2 "" H 4650 4650 50  0001 C CNN
+F 3 "" H 4650 4650 50  0001 C CNN
+	1    4650 4650
+	-1   0    0    1
+$EndComp
+$Comp
+L Device:C C9
+U 1 1 5BD38BD9
+P 6650 5800
+F 0 "C9" H 6765 5846 50  0000 L CNN
+F 1 "C" H 6765 5755 50  0000 L CNN
+F 2 "" H 6688 5650 50  0001 C CNN
+F 3 "~" H 6650 5800 50  0001 C CNN
+	1    6650 5800
+	1    0    0    -1
+$EndComp
+$Comp
+L power:+BATT #PWR021
+U 1 1 5BD38C4D
+P 6650 5650
+F 0 "#PWR021" H 6650 5500 50  0001 C CNN
+F 1 "+BATT" H 6665 5823 50  0000 C CNN
+F 2 "" H 6650 5650 50  0001 C CNN
+F 3 "" H 6650 5650 50  0001 C CNN
+	1    6650 5650
+	1    0    0    -1
+$EndComp
+$Comp
+L power:GNDD #PWR022
+U 1 1 5BD38CA8
+P 6650 5950
+F 0 "#PWR022" H 6650 5700 50  0001 C CNN
+F 1 "GNDD" H 6654 5795 50  0000 C CNN
+F 2 "" H 6650 5950 50  0001 C CNN
+F 3 "" H 6650 5950 50  0001 C CNN
+	1    6650 5950
+	1    0    0    -1
+$EndComp
 $EndSCHEMATC

Commit message: Specified footprints for decoupling caps
Parts:
- C6, C7, C8, C9: footprint (none) -> Capacitor_SMD:C_1206_3216Metric
- RV1: footprint uv1:Bourns_3269W -> Potentiometer_THT:Potentiometer_Bourns_3299W_Vertical
Changed lines of the file:
@@
 F 0 "RV1" H 4831 5046 50  0000 R CNN
 F 1 "20k" H 4831 4955 50  0000 R CNN
-F 2 "uv1:Bourns_3269W" H 4900 5000 50  0001 C CNN
+F 2 "Potentiometer_THT:Potentiometer_Bourns_3299W_Vertical" H 4900 5000 50  0001 C CNN
 F 3 "~" H 4900 5000 50  0001 C CNN
 	1    4900 5000
@@
 F 0 "C7" V 8098 3900 50  0000 C CNN
 F 1 "C" V 8189 3900 50  0000 C CNN
-F 2 "" H 8388 3750 50  0001 C CNN
+F 2 "Capacitor_SMD:C_1206_3216Metric" H 8388 3750 50  0001 C CNN
 F 3 "~" H 8350 3900 50  0001 C CNN
 	1    8350 3900
@@
 F 0 "C6" V 8048 1200 50  0000 C CNN
 F 1 "C" V 8139 1200 50  0000 C CNN
-F 2 "" H 8338 1050 50  0001 C CNN
+F 2 "Capacitor_SMD:C_1206_3216Metric" H 8338 1050 50  0001 C CNN
 F 3 "~" H 8300 1200 50  0001 C CNN
 	1    8300 1200
@@
 F 0 "C8" H 4765 4546 50  0000 L CNN
 F 1 "C" H 4765 4455 50  0000 L CNN
-F 2 "" H 4688 4350 50  0001 C CNN
+F 2 "Capacitor_SMD:C_1206_3216Metric" H 4688 4350 50  0001 C CNN
 F 3 "~" H 4650 4500 50  0001 C CNN
 	1    4650 4500
@@
 F 0 "C9" H 6765 5846 50  0000 L CNN
 F 1 "C" H 6765 5755 50  0000 L CNN
-F 2 "" H 6688 5650 50  0001 C CNN
+F 2 "Capacitor_SMD:C_1206_3216Metric" H 6688 5650 50  0001 C CNN
 F 3 "~" H 6650 5800 50  0001 C CNN
 	1    6650 5800

Commit message: Haven't committed in a while....
Parts:
- C2, C3, C4, C5, C6, C7, C8, C9: footprint Capacitor_SMD:C_1206_3216Metric -> Capacitor_SMD:C_0603_1608Metric
- R1, R2, R3, R4, R5: footprint Resistor_SMD:R_1206_3216Metric -> Resistor_SMD:R_0603_1608Metric
- U3: footprint Package_TO_SOT_SMD:SOT-23-5 -> Package_SO:SOIC-14_3.9x8.7mm_P1.27mm
- U4, U5: footprint Package_SO:TSSOP-16_4.4x5mm_P0.65mm -> Package_SO:SOIC-16_3.9x9.9mm_P1.27mm
Changed lines of the file:
@@
 F 0 "C4" V 3548 1050 50  0000 C CNN
 F 1 "0.1u" V 3639 1050 50  0000 C CNN
-F 2 "Capacitor_SMD:C_1206_3216Metric" H 3838 900 50  0001 C CNN
+F 2 "Capacitor_SMD:C_0603_1608Metric" H 3838 900 50  0001 C CNN
 F 3 "~" H 3800 1050 50  0001 C CNN
 	1    3800 1050
@@
 F 0 "R3" V 3593 6950 50  0000 C CNN
 F 1 "100k" V 3684 6950 50  0000 C CNN
-F 2 "Resistor_SMD:R_1206_3216Metric" V 3730 6950 50  0001 C CNN
+F 2 "Resistor_SMD:R_0603_1608Metric" V 3730 6950 50  0001 C CNN
 F 3 "~" H 3800 6950 50  0001 C CNN
 	1    3800 6950
@@
 F 0 "C5" V 3748 6600 50  0000 C CNN
 F 1 "100p" V 3839 6600 50  0000 C CNN
-F 2 "Capacitor_SMD:C_1206_3216Metric" H 4038 6450 50  0001 C CNN
+F 2 "Capacitor_SMD:C_0603_1608Metric" H 4038 6450 50  0001 C CNN
 F 3 "~" H 4000 6600 50  0001 C CNN
 	1    4000 6600
@@
 F 0 "C2" V 2548 4150 50  0000 C CNN
 F 1 "0.47u" V 2639 4150 50  0000 C CNN
-F 2 "Capacitor_SMD:C_1206_3216Metric" H 2838 4000 50  0001 C CNN
+F 2 "Capacitor_SMD:C_0603_1608Metric" H 2838 4000 50  0001 C CNN
 F 3 "~" H 2800 4150 50  0001 C CNN
 	1    2800 4150
@@
 F 0 "R1" H 2470 3946 50  0000 L CNN
 F 1 "47k" H 2470 3855 50  0000 L CNN
-F 2 "Resistor_SMD:R_1206_3216Metric" V 2330 3900 50  0001 C CNN
+F 2 "Resistor_SMD:R_0603_1608Metric" V 2330 3900 50  0001 C CNN
 F 3 "~" H 2400 3900 50  0001 C CNN
 	1    2400 3900
@@
 F 0 "R2" V 2243 2250 50  0000 C CNN
 F 1 "1M" V 2334 2250 50  0000 C CNN
-F 2 "Resistor_SMD:R_1206_3216Metric" V 2380 2250 50  0001 C CNN
+F 2 "Resistor_SMD:R_0603_1608Metric" V 2380 2250 50  0001 C CNN
 F 3 "~" H 2450 2250 50  0001 C CNN
 	1    2450 2250
@@
 F 0 "C3" H 2965 2496 50  0000 L CNN
 F 1 "0.01u" H 2965 2405 50  0000 L CNN
-F 2 "Capacitor_SMD:C_1206_3216Metric" H 2888 2300 50  0001 C CNN
+F 2 "Capacitor_SMD:C_0603_1608Metric" H 2888 2300 50  0001 C CNN
 F 3 "~" H 2850 2450 50  0001 C CNN
 	1    2850 2450
@@
 F 0 "R4" H 5320 4596 50  0000 L CNN
 F 1 "6.8k" H 5320 4505 50  0000 L CNN
-F 2 "Resistor_SMD:R_1206_3216Metric" V 5180 4550 50  0001 C CNN
+F 2 "Resistor_SMD:R_0603_1608Metric" V 5180 4550 50  0001 C CNN
 F 3 "~" H 5250 4550 50  0001 C CNN
 	1    5250 4550
@@
 F 0 "U4" H 7950 3328 50  0000 C CNN
 F 1 "74HC157" H 7950 3237 50  0000 C CNN
-F 2 "Package_SO:TSSOP-16_4.4x5mm_P0.65mm" H 7950 2250 50  0001 C CNN
+F 2 "Package_SO:SOIC-16_3.9x9.9mm_P1.27mm" H 7950 2250 50  0001 C CNN
 F 3 "http://www.ti.com/lit/gpn/sn74LS157" H 7950 2250 50  0001 C CNN
 	1    7950 2250
@@
 F 0 "U5" H 7950 5878 50  0000 C CNN
 F 1 "74HC157" H 7950 5787 50  0000 C CNN
-F 2 "Package_SO:TSSOP-16_4.4x5mm_P0.65mm" H 7950 4800 50  0001 C CNN
+F 2 "Package_SO:SOIC-16_3.9x9.9mm_P1.27mm" H 7950 4800 50  0001 C CNN
 F 3 "http://www.ti.com/lit/gpn/sn74LS157" H 7950 4800 50  0001 C CNN
 	1    7950 4800
@@
 F 0 "R5" H 6220 2546 50  0000 L CNN
 F 1 "470k" H 6220 2455 50  0000 L CNN
-F 2 "Resistor_SMD:R_1206_3216Metric" V 6080 2500 50  0001 C CNN
+F 2 "Resistor_SMD:R_0603_1608Metric" V 6080 2500 50  0001 C CNN
 F 3 "~" H 6150 2500 50  0001 C CNN
 	1    6150 2500
@@
 F 0 "U3" H 6675 5467 50  0000 C CNN
 F 1 "74AHC1G04" H 6675 5376 50  0000 C CNN
-F 2 "Package_TO_SOT_SMD:SOT-23-5" H 6700 5200 50  0001 C CNN
+F 2 "Package_SO:SOIC-14_3.9x8.7mm_P1.27mm" H 6700 5200 50  0001 C CNN
 F 3 "http://www.ti.com/lit/sg/scyt129e/scyt129e.pdf" H 6700 5200 50  0001 C CNN
 	1    6700 5200
@@
 F 0 "C7" V 8098 3900 50  0000 C CNN
 F 1 "C" V 8189 3900 50  0000 C CNN
-F 2 "Capacitor_SMD:C_1206_3216Metric" H 8388 3750 50  0001 C CNN
+F 2 "Capacitor_SMD:C_0603_1608Metric" H 8388 3750 50  0001 C CNN
 F 3 "~" H 8350 3900 50  0001 C CNN
 	1    8350 3900
@@
 F 0 "C6" V 8048 1200 50  0000 C CNN
 F 1 "C" V 8139 1200 50  0000 C CNN
-F 2 "Capacitor_SMD:C_1206_3216Metric" H 8338 1050 50  0001 C CNN
+F 2 "Capacitor_SMD:C_0603_1608Metric" H 8338 1050 50  0001 C CNN
 F 3 "~" H 8300 1200 50  0001 C CNN
 	1    8300 1200
@@
 F 0 "C8" H 4765 4546 50  0000 L CNN
 F 1 "C" H 4765 4455 50  0000 L CNN
-F 2 "Capacitor_SMD:C_1206_3216Metric" H 4688 4350 50  0001 C CNN
+F 2 "Capacitor_SMD:C_0603_1608Metric" H 4688 4350 50  0001 C CNN
 F 3 "~" H 4650 4500 50  0001 C CNN
 	1    4650 4500
@@
 F 0 "C9" H 6765 5846 50  0000 L CNN
 F 1 "C" H 6765 5755 50  0000 L CNN
-F 2 "Capacitor_SMD:C_1206_3216Metric" H 6688 5650 50  0001 C CNN
+F 2 "Capacitor_SMD:C_0603_1608Metric" H 6688 5650 50  0001 C CNN
 F 3 "~" H 6650 5800 50  0001 C CNN
 	1    6650 5800
