File: uv1.sch (KiCad schematic (older format))
At the start: 25 parts, among them J1 Conn_02x07_Odd_Even, J2 - +, SW1 SW_Push, U1 TC7106, U2 DE115-RS-20, U3 74AHC1G04, U4 74HC157, U5 74HC157

Commit message: Removed last digit enable logic from uv1.sch
Parts:
- removed C6, C7, C9: C, Capacitor_SMD:C_0603_1608Metric, symbol Device:C
- removed JP1: Jumper_NO_Small, Connector_PinHeader_1.27mm:PinHeader_1x02_P1.27mm_Vertical, symbol Device:Jumper_NO_Small
- removed R5: 470k, Resistor_SMD:R_0603_1608Metric, symbol Device:R
- removed U4, U5: 74HC157, Package_SO:SOIC-16_3.9x9.9mm_P1.27mm, symbol 74xx:74LS157
- C8: value C -> 0.1u
Connections:
- net labels removed: DIGIT3_EN, MUX_3A, MUX_3B, MUX_3C, MUX_3D, MUX_3E, MUX_3F, MUX_3G
- wire segments 171 -> 130
Other:
- moved on the sheet: U3
