File: uv1.kicad_pcb (KiCad board)
At the start: 2 copper layers, 54.9 x 63 mm, 25 parts, among them J1 Conn_02x07_Odd_Even, J2 - +, SW1 SW_Push, U1 TC7106, U2 DE115-RS-20, U3 74AHC1G04, U4 74HC157, U5 74HC157

Commit message: Before changing gate packages
Parts:
- moved R5 2.64 mm to (116.0, 84.7)
- moved JP1 2.48 mm to (120.0, 84.7)
Routing:
- net +BATT: track 127.7 -> 126.9 mm
- added copper zone on B.Cu, net /ACOM
- added copper zone on F.Cu, net /ACOM
- added copper zone on F.Cu, net GND

Commit message: Haven't committed in a while....
Parts:
- C2, C3, C4, C5, C6, C7, C8, C9: footprint Capacitor_SMD:C_1206_3216Metric -> Capacitor_SMD:C_0603_1608Metric
- R1, R2, R3, R4, R5: footprint Resistor_SMD:R_1206_3216Metric -> Resistor_SMD:R_0603_1608Metric
- U3: footprint Package_TO_SOT_SMD:SOT-23-5 -> Package_SO:SOIC-14_3.9x8.7mm_P1.27mm
- U4, U5: footprint Package_SO:TSSOP-16_4.4x5mm_P0.65mm -> Package_SO:SOIC-16_3.9x9.9mm_P1.27mm
- moved R5 42.0 mm to (117.8, 126.7)
- moved JP1 42.0 mm to (121.0, 126.7)
- moved R1 38.4 mm to (77.0, 92.0), turned to 90 degrees
- moved C8 36.5 mm to (80.5, 107.5), turned to 90 degrees
- moved C2 35.7 mm to (80.0, 92.0), turned to 90 degrees
- moved C1 33.1 mm to (84.0, 89.0), turned to 270 degrees
- moved C9 9.34 mm to (109.2, 119.4), turned to 180 degrees
- moved R3 6.86 mm to (91.7, 118.9)
- moved C5 6.07 mm to (87.1, 118.9)
- moved U3 5.85 mm to (117.8, 109.2), turned to 270 degrees
- moved U1 5.29 mm to (89.0, 109.2)
- moved C7 4.79 mm to (117.8, 103.9), turned to 180 degrees
- moved C3 4.39 mm to (80.5, 110.8)
- moved RV1 3.00 mm to (116.0, 134.0), turned to 90 degrees
- moved C4 2.86 mm to (80.5, 114.1)
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Connections:
- J1 pad 10: Net-(J1-Pad10) -> (no net)
- J1 pad 5: Net-(J1-Pad5) -> (no net)
- J1 pad 6: Net-(J1-Pad6) -> (no net)
- J1 pad 7: Net-(J1-Pad7) -> (no net)
- J1 pad 8: Net-(J1-Pad8) -> (no net)
- J1 pad 9: Net-(J1-Pad9) -> (no net)
Routing:
- net -BATT: track 106.5 -> 33.2 mm
- net Net-(C1-Pad1): track 66.7 -> 7.92 mm
- net Net-(C3-Pad1): track 12.8 -> 53.8 mm
- net Net-(C8-Pad1): track 66.2 -> 43.1 mm, vias 1 -> 2
- net +BATT: track 126.9 -> 147.8 mm, vias 0 -> 1
- net /ACOM: track 115.1 -> 133.6 mm
- net Net-(R1-Pad1): track 38.9 -> 21.0 mm
- net Net-(RV1-Pad2): track 38.1 -> 55.6 mm, vias 1 -> 0
- net Net-(C1-Pad2): track 33.2 -> 17.2 mm
- net GND: track 59.3 -> 74.7 mm, vias 5 -> 4
- net /LCD_BP: track 126.8 -> 141.1 mm, vias 1 -> 3
- net /MUX_3E: track 7.70 -> 20.7 mm, vias 0 -> 2
- net Net-(U3-Pad4): track 7.21 -> 19.5 mm
- net /DIGIT3_EN: track 39.5 -> 51.4 mm, vias 2 -> 0
- net /LCD_1A: track 12.9 -> 23.1 mm, vias 1 -> 0
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- removed copper zone on B.Cu, net /ACOM
- removed copper zone on F.Cu, net /ACOM
- removed copper zone on F.Cu, net GND

Commit message: Routed
Parts:
- removed C6, C7, C9: C, Capacitor_SMD:C_0603_1608Metric
- removed JP1: Jumper_NO_Small, Connector_PinHeader_1.27mm:PinHeader_1x02_P1.27mm_Vertical
- removed R5: 470k, Resistor_SMD:R_0603_1608Metric
- removed U4, U5: 74HC157, Package_SO:SOIC-16_3.9x9.9mm_P1.27mm
- C8: value C -> 0.1u
- moved C2 23.6 mm to (76.0, 115.2)
- moved C1 19.7 mm to (76.0, 107.0), turned to 90 degrees
- moved R1 19.0 mm to (76.8, 111.0), turned to 180 degrees
- moved C4 8.05 mm to (88.0, 117.0)
- moved U1 7.00 mm to (96.0, 109.0)
- moved R3 6.37 mm to (98.0, 118.0), turned to 90 degrees
- moved C5 5.92 mm to (93.0, 118.0), turned to 90 degrees
- moved U3 5.81 mm to (112.0, 109.0), turned to 90 degrees
- moved D1 5.64 mm to (86.0, 130.0)
- moved C3 5.02 mm to (85.0, 113.0), turned to 0 degrees
- moved C8 4.73 mm to (85.0, 106.0)
- moved R2 3.50 mm to (84.0, 102.0), turned to 0 degrees
Connections:
- U1 pad 2: /MUX_3D -> /LCD_3D
- U1 pad 3: /MUX_3C -> /LCD_3C
- U1 pad 4: /MUX_3B -> /LCD_3B
- U1 pad 5: /MUX_3A -> /LCD_3A
- U1 pad 6: /MUX_3F -> /LCD_3F
- U1 pad 7: /MUX_3G -> /LCD_3G
- U1 pad 8: /MUX_3E -> /LCD_3E
- U3 pad 4: Net-(U3-Pad4) -> /LCD_DP3
Routing:
- net /LCD_BP: track 141.1 -> 81.0 mm, vias 3 -> 2
- net /DIGIT3_EN: track 51.4 -> 0.00 mm
- net GND: track 74.7 -> 25.7 mm, vias 4 -> 2
- net +BATT: track 147.8 -> 99.4 mm, vias 1 -> 0
- net /ACOM: track 133.6 -> 87.6 mm
- net Net-(C3-Pad1): track 53.8 -> 16.1 mm, vias 0 -> 2
- net Net-(C8-Pad1): track 43.1 -> 70.6 mm, vias 2 -> 1
- net /MUX_3E: track 20.7 -> 0.00 mm, vias 2 -> 0
- net Net-(U3-Pad4): track 19.5 -> 0.00 mm
- net Net-(RV1-Pad2): track 55.6 -> 37.7 mm, vias 0 -> 1
- net /MUX_3G: track 16.6 -> 0.00 mm, vias 2 -> 0
- net /LCD_2E: track 22.2 -> 38.2 mm
- net /MUX_3A: track 14.8 -> 0.00 mm
- net /MUX_3C: track 14.2 -> 0.00 mm
- net -BATT: track 33.2 -> 46.3 mm, vias 1 -> 0
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